File: hardware/servo.kicad_pcb (KiCad board)
At the start: 4 copper layers, 40 x 40 mm, 113 parts, among them J1 DRILL, J10 CON-SERVO, J2 DRILL, J3 DRILL, J4 DRILL, J5 USB-MINI-B-SMD, J6 STACK-UP-HIGH, J7 STACK-DOWN, J8 STACK-UP-HIGH, J9 STACK-DOWN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

Commit message: Add 3d information (final)
Parts:
- C1, C10, C12, C13, C14, C15, C16, C18, C2, C20, C21, C25, C26, C27, C28, C32, C5, C8, C9: footprint 0402 -> kicad-libraries:C0402
- C11, C19, C24, C30, C7, FB1, FB2, FB3, FB4, FB5, R9: footprint 0603 -> kicad-libraries:C0603
- C17, C4, C6, L2: footprint 0805 -> kicad-libraries:C0805
- C22: footprint ELKO_83 -> kicad-libraries:ELKO_83
- C23, C31: footprint 1206 -> kicad-libraries:C1206
- C29: footprint 0402 -> kicad-libraries:0402
- C3: footprint 3528-21 -> kicad-libraries:3528-21
- C33: footprint 7343 -> kicad-libraries:7343
- D1, D2: footprint D0603 -> kicad-libraries:D0603
- D3, D4, D5, D6: footprint SOD-123 -> kicad-libraries:SOD-123
- D7, D8, D9: footprint SOD-128 -> kicad-libraries:SOD-128
- Fiducial_Mark (x4): footprint Fiducial_Mark -> kicad-libraries:Fiducial_Mark
- J1, J2, J3, J4: footprint DRILL_NP -> kicad-libraries:DRILL_NP
- J10: footprint CON-Servo -> kicad-libraries:CON-Servo
- J5: footprint USB-MINI-B-SMD -> kicad-libraries:USB-MINI-B-SMD
- J6, J8: footprint BTB08-ACS-TOP -> kicad-libraries:BTB08-ACS-TOP
- J7, J9: footprint BTB08-ACS-BTM -> kicad-libraries:BTB08-ACS-BTM
- L1: footprint NR3030 -> kicad-libraries:NR3030
- L3: footprint SRP7030 -> kicad-libraries:SRP7030
- P1, P2: footprint CON-SENSOR -> kicad-libraries:CON-SENSOR
- P3: footprint OQ_2P -> kicad-libraries:OQ_2P
- Q1, Q2: footprint SOIC-8-MOSFET -> kicad-libraries:SOIC-8-MOSFET
- Q3: footprint SOT23GDS -> kicad-libraries:SOT23GDS
- R1, R10, R11, R12, R13, R14, R15, R16, R17, R18, R19, R2, R20, R21, R22, R23, R3, R4, R7, R8: footprint 0402 -> kicad-libraries:R0402
- R24, R25, R26, R27, R28, R29, R30: footprint 0805 -> kicad-libraries:R0805
- R5, R6: footprint 0603 -> kicad-libraries:R0603
- RP1, RP2: footprint 4X0603 -> kicad-libraries:4X0603
- SW1, SW2: footprint TACT-SWITCH -> kicad-libraries:TACT-SWITCH
- U1: footprint LQFP64 -> kicad-libraries:LQFP64
- U2: footprint SOT23-5 -> kicad-libraries:SOT23-5
- U3: footprint SO-8 -> kicad-libraries:SO-8
- U4: footprint TSSOP20 -> kicad-libraries:TSSOP20
- U5: footprint SOIC16 -> kicad-libraries:SOIC16
- VAL: footprint CE_5mm -> kicad-libraries:CE_5mm
- VAL: footprint WEEE_7mm -> kicad-libraries:WEEE_7mm
- X1: footprint CRYSTAL_3225 -> kicad-libraries:CRYSTAL_3225
- turned R12 to 0 degrees
Connections:
- D6 pad 2: N-00000127 -> Net-(D6-Pad2)
- D7 pad 1: N-00000128 -> Net-(D7-Pad1)
- P3 pad 1: N-00000128 -> Net-(D7-Pad1)
- Q1 pad G: N-00000127 -> Net-(D6-Pad2)
- R12 pad 1: N-00000127 -> Net-(D7-Pad1)
- R12 pad 2: N-00000128 -> Net-(D6-Pad2)
- R14 pad 2: N-00000128 -> Net-(D7-Pad1)
Routing:
- net Net-(D7-Pad1): track 0.00 -> 12.2 mm
- net N-00000128: track 12.2 -> 0.00 mm
- net Net-(D6-Pad2): track 0.00 -> 8.95 mm, vias 0 -> 1
- net N-00000127: track 8.95 -> 0.00 mm, vias 1 -> 0
